File: hardware/rp-micro.kicad_pcb (KiCad board)
At the start: 2 copper layers, 17.8 x 33 mm, 46 parts, among them J1 USB_C_Receptacle_USB2.0, J2 Conn_01x12, J3 Conn_01x12, J4 Conn_01x05, SW1 BOOT, SW2 RESET, U1 RT9013-33GB, U2 W25Q16JVUXIQ, U3 RP2040, Y1 12MHz

Commit message: Update track
Parts:
- renumbered C3 to C1, C17 to C10, C8 to C11, C9 to C12, C10 to C13, C11 to C14, C12 to C15, C13 to C16, C14 to C17, C1 to C2, C2 to C3, C15 to C8, C16 to C9, R11 to R10, R12 to R11, R9 to R12, R3 to R2, R4 to R3, R5 to R4, R2 to R5, R10 to R9
Routing:
- net GND: vias 34 -> 35
